File: kicad/bitdoglabsmd/bitdoglab_smd.kicad_sch (KiCad schematic)
At the start: 139 parts, among them J1 Conn_01x03, J10 3V3, J11 5V-VSYS, J12 Conn_01x05_Pin, J13 Conn_01x05_Pin, J14 Conn_01x01_Socket, J15 0, J16 1, J17 2, J18 3, J19 JOYSTICK, J2 conector_idc, J20 Conn_01x04_Pin, J21 Conn_01x04_Pin, J5 Conn_01x05_Pin, J6 Conn_01x05_Pin, J7 GND, J8 ANA-IN, J9 GND, Q1 BC817, Q2 BC817, Q4 CMA-4544PF-W, Q5 DMG2305UX-13, SW1 Reset, SW2 Botão, SW3 Button_B, U2 MAX4466EXK+T, U3 IP5306

Commit message: BitDogLab SMD version 5.2
Parts:
- removed J14: Conn_01x01_Socket, Connector_PinHeader_2.54mm:PinHeader_1x01_P2.54mm_Vertical, symbol Connector:Conn_01x01_Socket
- added BZ2, BZ4: Buzzer_B_SMD, Buzzer_Beeper:MagneticBuzzer_CUI_CMT-8504-100-SMT, symbol Device:Buzzer
- added J3: Conn_01x02, Connector_PinHeader_2.54mm:PinHeader_1x02_P2.54mm_Vertical, symbol Connector_Generic:Conn_01x02
Connections:
- net GNDREF: now also J3.2 (Pin_2)
- net VSYS: now also BZ2.1 (-), BZ4.1 (-)
- net at BZ3.2 (+), Q2.3 (C): now also BZ4.2 (+)
- net at BZ1.2 (+), Q1.3 (C): now also BZ2.2 (+)
- net at D28.2 (DOUT): now also J3.1 (Pin_1)
Changed lines of the file:
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@@
   (title_block
     (title "BitDogLab SMD version")
-    (date "2024-02-22")
-    (rev "v5.1")
+    (date "2024-02-26")
+    (rev "v5.2")
     (company "Universidade Estadual de Campinas (Unicamp)*/Hardware Innovation Technologies (HwIT)**")
     (comment 1 "Juliano Rodrigues Fernandes de Oliveira**")
@@
   (junction (at 381 109.855) (diameter 0) (color 0 0 0 0)
   )
+  (junction (at 212.09 200.66) (diameter 0) (color 0 0 0 0)
+  )
   (junction (at 307.34 238.76) (diameter 0) (color 0 0 0 0)
   )
@@
   (junction (at 381 179.07) (diameter 0) (color 0 0 0 0)
   )
+  (junction (at 212.09 227.33) (diameter 0) (color 0 0 0 0)
+  )
   (junction (at 370.84 231.14) (diameter 0) (color 0 0 0 0)
   )
@@
   (junction (at 381 85.09) (diameter 0) (color 0 0 0 0)
   )
+  (junction (at 203.454 195.58) (diameter 0) (color 0 0 0 0)
+  )
   (junction (at 63.5 66.04) (diameter 0) (color 0 0 0 0)
   )
@@
   (junction (at 381 139.7) (diameter 0) (color 0 0 0 0)
   )
+  (junction (at 204.216 222.25) (diameter 0) (color 0 0 0 0)
+  )
   (junction (at 355.6 179.07) (diameter 0) (color 0 0 0 0)
   )
@@
     (stroke (width 0) (type default))
   )
-  (wire (pts (xy 196.85 195.58) (xy 212.09 195.58))
+  (wire (pts (xy 394.208 173.99) (xy 390.906 173.99))
+    (stroke (width 0) (type default))
+  )
+  (wire (pts (xy 196.85 195.58) (xy 203.454 195.58))
     (stroke (width 0) (type default))
   )
@@
     (stroke (width 0) (type default))
   )
+  (wire (pts (xy 212.09 208.534) (xy 203.454 208.534))
+    (stroke (width 0) (type default))
+  )
   (wire (pts (xy 146.05 38.1) (xy 154.94 38.1))
     (stroke (width 0.254) (type default))
@@
     (stroke (width 0.254) (type default))
   )
-  (wire (pts (xy 388.62 171.45) (xy 390.525 171.45))
+  (wire (pts (xy 388.62 171.45) (xy 394.208 171.45))
     (stroke (width 0) (type default))
   )
@@
     (stroke (width 0) (type default))
   )
+  (wire (pts (xy 203.454 195.58) (xy 212.09 195.58))
+    (stroke (width 0) (type default))
+  )
   (wire (pts (xy 288.29 99.06) (xy 298.45 99.06))
     (stroke (width 0) (type default))
@@
     (stroke (width 0) (type default))
   )
+  (wire (pts (xy 204.216 222.25) (xy 212.09 222.25))
+    (stroke (width 0) (type default))
+  )
   (wire (pts (xy 373.38 109.855) (xy 373.38 111.76))
     (stroke (width 0) (type default))
@@
     (stroke (width 0) (type default))
   )
-  (wire (pts (xy 196.85 222.25) (xy 212.09 222.25))
+  (wire (pts (xy 196.85 222.25) (xy 204.216 222.25))
     (stroke (width 0) (type default))
   )
@@
     (stroke (width 0) (type default))
   )
+  (wire (pts (xy 203.454 208.534) (xy 203.454 195.58))
+    (stroke (width 0) (type default))
+  )
   (wire (pts (xy 283.21 231.14) (xy 285.75 231.14))
     (stroke (width 0) (type default))
@@
     (stroke (width 0) (type default))
   )
+  (wire (pts (xy 390.906 173.99) (xy 390.906 177.8))
+    (stroke (width 0) (type default))
+  )
   (wire (pts (xy 361.315 202.565) (xy 361.315 207.01))
     (stroke (width 0) (type default))
@@
     (stroke (width 0) (type default))
   )
+  (wire (pts (xy 212.09 235.458) (xy 204.216 235.458))
+    (stroke (width 0) (type default))
+  )
   (wire (pts (xy 105.41 218.44) (xy 116.205 218.44))
     (stroke (width 0) (type default))
@@
     (stroke (width 0) (type default))
   )
+  (wire (pts (xy 212.09 200.66) (xy 212.09 203.454))
+    (stroke (width 0) (type default))
+  )
   (wire (pts (xy 156.21 223.52) (xy 162.56 223.52))
     (stroke (width 0) (type default))
@@
     (stroke (width 0) (type default))
   )
+  (wire (pts (xy 212.09 227.33) (xy 212.09 230.378))
+    (stroke (width 0) (type default))
+  )
   (wire (pts (xy 363.22 171.45) (xy 373.38 171.45))
     (stroke (width 0) (type default))
@@
     (stroke (width 0) (type default))
   )
+  (wire (pts (xy 204.216 235.458) (xy 204.216 222.25))
+    (stroke (width 0) (type default))
+  )
   (wire (pts (xy 60.96 200.66) (xy 60.96 203.2))
     (stroke (width 0) (type default))
@@
     )
   )
+  (symbol (lib_name "GNDREF_4") (lib_id "power:GNDREF") (at 390.906 177.8 0) (unit 1)
+    (in_bom yes) (on_board yes) (dnp no)
+    (property "Reference" "#PWR055" (at 390.906 184.15 0)
+      (effects (font (size 1.27 1.27)) hide)
+    )
+    (property "Value" "GNDREF" (at 395.986 180.34 0)
+      (effects (font (size 1.27 1.27)) hide)
+    )
+    (property "Footprint" "" (at 390.906 177.8 0)
+      (effects (font (size 1.27 1.27)) hide)
+    )
+    (property "Datasheet" "" (at 390.906 177.8 0)
+      (effects (font (size 1.27 1.27)) hide)
+    )
+    (pin "1")
+    (instances
+      (project "bitdoglab_smd"
+        (path "/09159d3e-7c55-4754-a166-a35b245d09f3"
+          (reference "#PWR055") (unit 1)
+        )
+      )
+    )
+  )
   (symbol (lib_id "power:+3.3V") (at 394.716 212.344 180) (unit 1)
     (in_bom yes) (on_board yes) (dnp no) (fields_autoplaced)
@@
     )
   )
+  (symbol (lib_id "Device:Buzzer") (at 214.63 205.994 0) (unit 1)
+    (in_bom yes) (on_board yes) (dnp no) (fields_autoplaced)
+    (property "Reference" "BZ2" (at 218.44 204.724 0)
+      (effects (font (size 1.27 1.27)) (justify left))
+    )
+    (property "Value" "Buzzer_B_SMD" (at 218.44 207.264 0)
+      (effects (font (size 1.27 1.27)) (justify left))
+    )
+    (property "Footprint" "Buzzer_Beeper:MagneticBuzzer_CUI_CMT-8504-100-SMT" (at 213.995 203.454 90)
+      (effects (font (size 1.27 1.27)) hide)
+    )
+    (property "Datasheet" "~" (at 213.995 203.454 90)
+      (effects (font (size 1.27 1.27)) hide)
+    )
+    (pin "1")
+    (pin "2")
+    (instances
+      (project "bitdoglab_smd"
+        (path "/09159d3e-7c55-4754-a166-a35b245d09f3"
+          (reference "BZ2") (unit 1)
+        )
+      )
+    )
+  )
   (symbol (lib_id "Device:L_Small") (at 110.49 40.64 90) (unit 1)
     (in_bom yes) (on_board yes) (dnp no)
@@
     )
   )
+  (symbol (lib_id "Connector_Generic:Conn_01x02") (at 399.288 171.45 0) (unit 1)
+    (in_bom yes) (on_board yes) (dnp no) (fields_autoplaced)
+    (property "Reference" "J3" (at 401.32 171.45 0)
+      (effects (font (size 1.27 1.27)) (justify left))
+    )
+    (property "Value" "Conn_01x02" (at 401.32 173.99 0)
+      (effects (font (size 1.27 1.27)) (justify left))
+    )
+    (property "Footprint" "Connector_PinHeader_2.54mm:PinHeader_1x02_P2.54mm_Vertical" (at 399.288 171.45 0)
+      (effects (font (size 1.27 1.27)) hide)
+    )
+    (property "Datasheet" "~" (at 399.288 171.45 0)
+      (effects (font (size 1.27 1.27)) hide)
+    )
+    (pin "1")
+    (pin "2")
+    (instances
+      (project "bitdoglab_smd"
+        (path "/09159d3e-7c55-4754-a166-a35b245d09f3"
+          (reference "J3") (unit 1)
+        )
+      )
+    )
+  )
   (symbol (lib_id "Device:LED_RGB") (at 183.515 100.33 0) (unit 1)
     (in_bom yes) (on_board yes) (dnp no) (fields_autoplaced)
@@
     )
   )
+  (symbol (lib_id "Device:Buzzer") (at 214.63 232.918 0) (unit 1)
+    (in_bom yes) (on_board yes) (dnp no) (fields_autoplaced)
+    (property "Reference" "BZ4" (at 218.44 231.648 0)
+      (effects (font (size 1.27 1.27)) (justify left))
+    )
+    (property "Value" "Buzzer_B_SMD" (at 218.44 234.188 0)
+      (effects (font (size 1.27 1.27)) (justify left))
+    )
+    (property "Footprint" "Buzzer_Beeper:MagneticBuzzer_CUI_CMT-8504-100-SMT" (at 213.995 230.378 90)
+      (effects (font (size 1.27 1.27)) hide)
+    )
+    (property "Datasheet" "~" (at 213.995 230.378 90)
+      (effects (font (size 1.27 1.27)) hide)
+    )
+    (pin "1")
+    (pin "2")
+    (instances
+      (project "bitdoglab_smd"
+        (path "/09159d3e-7c55-4754-a166-a35b245d09f3"
+          (reference "BZ4") (unit 1)
+        )
+      )
+    )
+  )
   (symbol (lib_id "LED:WS2812B") (at 381 124.46 0) (unit 1)
     (in_bom yes) (on_board yes) (dnp no) (fields_autoplaced)
@@
         )
       )
-    )
-  )
-  (symbol (lib_id "Connector:Conn_01x01_Socket") (at 395.605 171.45 0) (unit 1)
-    (in_bom yes) (on_board yes) (dnp no) (fields_autoplaced)
-    (property "Reference" "J14" (at 397.51 170.18 0)
-      (effects (font (size 1.27 1.27)) (justify left))
-    )
-    (property "Value" "Conn_01x01_Socket" (at 397.51 172.72 0)
-      (effects (font (size 1.27 1.27)) (justify left))
-    )
-    (property "Footprint" "Connector_PinHeader_2.54mm:PinHeader_1x01_P2.54mm_Vertical" (at 395.605 171.45 0)
-      (effects (font (size 1.27 1.27)) hide)
-    )
-    (property "Datasheet" "~" (at 395.605 171.45 0)
-      (effects (font (size 1.27 1.27)) hide)
-    )
-    (pin "1")
-    (instances
-      (project "bitdoglab_smd"
-        (path "/09159d3e-7c55-4754-a166-a35b245d09f3"
-          (reference "J14") (unit 1)
-        )
-      )
