File: kicad/bitdoglab_v5_0/bitdoglab_v5.kicad_pcb (KiCad board)
At the start: 2 copper layers, 87.9 x 123.9 mm, 76 parts, among them J1 Conn_01x20_Socket, J10 3V3, J11 5V-VSYS, J12 Conn_01x05_Pin, J13 Conn_01x05_Pin, J14 5x5 Matrix led, J15 0, J16 1, J17 2, J18 3, J19 JOYSTICK, J2 conector_idc, J20 JST_EH_B4B-EH-A_1x04_P2.50mm_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, J21 JST_EH_B4B-EH-A_1x04_P2.50mm_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, J3 Conn_01x20_Socket, J4 jumper_mic, J5 Conn_01x05_Pin, J6 Conn_01x05_Pin, J7 GND, J8 ANA-IN, J9 GND, Q1 DMG2305UX-13, Q2 BC337, Q3 BC337, SW1 Reset, SW2 Botão, SW3 Button_B, U1 3.3v_tht, U4 MIC

Commit message: Sincronizacao da placa com o esquemático
Parts:
- removed ? (x6): , 
- added C3: C_pth, Capacitor_THT:CP_Radial_D5.0mm_P2.50mm, F.Cu at (172.5, 140.0)
- added C4: C_pth, Capacitor_THT:CP_Radial_D5.0mm_P2.50mm, F.Cu at (149.0, 143.7)
- added R_pulldown1: 10k, Resistor_THT:R_Axial_DIN0207_L6.3mm_D2.5mm_P7.62mm_Horizontal, B.Cu at (124.1, 134.0)
- C1, C2: value C_Polarized_Small -> C_smd
- D1: value LED_RGB -> LED_RGB_SMD
- D3: value Zener -> 1N5231
- D4: value D Shot -> D_Schottky
- J20, J21: value JST_EH_B4B-EH-A_1x04_P2.50mm_Vertical -> Conn_01x04_Pin
- gave numbers to parts that had none: 13
- renumbered REF** to JOY1, A1 to pico1, a102 to solar01
Connections:
- BT1 pad 1: Net-(BT1-+) -> V_BAT +
- CARGA_SOLAR1 pad 2: Solar-in -> Net-(CARGA_SOLAR1-Pin_2)
- Charge_DisCharge1 pad 1: Net-(Q1-D) -> Net-(Charge_DisCharge1-OUT5V)
- Charge_DisCharge1 pad 3: Net-(BT1-+) -> V_BAT +
- D2 pad 1: Net-(D2-RA) -> Net-(D1-RA)
- D2 pad 3: Net-(D2-BA) -> Net-(D1-BA)
- D2 pad 4: Net-(D2-GA) -> Net-(D1-GA)
- D3 pad 1: (no net) -> Net-(D3-K)
- D3 pad 2: (no net) -> GNDREF
- D4 pad 2: (no net) -> Net-(D3-K)
- J2 pad 4: /GP10 -> /GP08
- J2 pad 8: /GP08 -> /GP04
- Q1 pad 3: Net-(Charge DisCharge1-OUT5V) -> Net-(Charge_DisCharge1-OUT5V)
- R2 pad 1: /GP04 -> /GP10
- R_1W1 pad 1: Solar-in -> Net-(D3-K)
- R_1W1 pad 2: (no net) -> Net-(CARGA_SOLAR1-Pin_2)
- Rb_150 pad 1: Net-(D2-BA) -> Net-(D1-BA)
- Rg_220 pad 1: Net-(D2-GA) -> Net-(D1-GA)
- Rr_220 pad 1: Net-(D2-RA) -> Net-(D1-RA)
- V_BAT1 pad 2: Net-(BT1-+) -> V_BAT +
Routing:
- net VSYS: track 302.5 -> 0.00 mm, vias 6 -> 0
- net +3.3V: track 282.7 -> 0.00 mm, vias 2 -> 0
- net 3.3_OUT: track 153.9 -> 0.00 mm, vias 3 -> 0
- net /GP28: track 116.2 -> 0.00 mm
- net VBUS: track 105.4 -> 0.00 mm
- net /pino_31: track 68.5 -> 0.00 mm
- net /pino_07: track 66.7 -> 0.00 mm, vias 3 -> 0
- net /GP08: track 61.1 -> 0.00 mm
- net /GP09: track 60.3 -> 0.00 mm
- net /pino_29: track 59.7 -> 0.00 mm
- net /GP03: track 56.9 -> 0.00 mm
- net /pino_32: track 56.8 -> 0.00 mm
- net /GP10: track 55.1 -> 0.00 mm
- net /GP20: track 49.8 -> 0.00 mm
- net /GP02: track 49.4 -> 0.00 mm
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Other:
- board text added: "V 5.4"
- board text removed: "C1"
- board text removed: "C2"
- board text removed: "Diodo Shot"
- board text removed: "V 5"
- board text removed: "Zener 1N5231 A C"
