File: kicad/bitdoglab_v5_0/bitdoglab_v5.kicad_sch (KiCad schematic)
At the start: 52 parts, among them J1 Conn_01x20_Socket, J10 3V3, J11 5V-VSYS, J12 Conn_01x05_Pin, J13 Conn_01x05_Pin, J14 5x5 Matrix led, J15 0, J16 1, J17 2, J18 3, J19 JOYSTICK, J2 conector_idc, J20 Conn_01x04_Pin, J21 Conn_01x04_Pin, J3 Conn_01x20_Socket, J4 jumper_mic, J5 Conn_01x05_Pin, J6 Conn_01x05_Pin, J7 GND, J8 ANA-IN, J9 GND, Q1 DMG2305UX-13, Q2 BC337, Q3 BC337, SW1 Reset, SW2 Botão, SW3 Button_B, U1 3.3v_tht, U4 MIC

Commit message: Sincronizacao da placa com o esquemático
Parts:
- added C3, C4: C_pth, Capacitor_THT:CP_Radial_D5.0mm_P2.50mm, symbol Device:C_Polarized_Small
- added R_pulldown1: 10k, Resistor_THT:R_Axial_DIN0207_L6.3mm_D2.5mm_P7.62mm_Horizontal, symbol Device:R
- C1, C2: value C_Polarized_Small -> C_smd
- renumbered A1 to pico1
Connections:
- net +3.3V: now also C4.1
- net GNDREF: now also C3.2, C4.2, R_pulldown1.2
- net GP04: now also J2.8 (Pin_8); no longer R2.1
- net GP08: now also J2.4 (Pin_4); no longer J2.8 (Pin_8)
- net GP10: now also R2.1; no longer J2.4 (Pin_4)
- net VBUS: now also R_pulldown1.1
- net VSYS: now also C3.1
Changed lines of the file:
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@@
   (junction (at 254 135.89) (diameter 0) (color 0 0 0 0)
   )
+  (junction (at 38.1 40.64) (diameter 0) (color 0 0 0 0)
+  )
   (junction (at 105.41 39.37) (diameter 0) (color 0 0 0 0)
   )
   (junction (at 25.4 83.82) (diameter 0) (color 0 0 0 0)
   )
+  (junction (at 123.19 39.37) (diameter 0) (color 0 0 0 0)
+  )
   (junction (at 212.09 114.3) (diameter 0) (color 0 0 0 0)
   )
@@
   (junction (at 48.26 40.64) (diameter 0) (color 0 0 0 0)
   )
+  (junction (at 58.42 40.64) (diameter 0) (color 0 0 0 0)
+  )
   (wire (pts (xy 118.11 148.59) (xy 121.92 148.59))
     (stroke (width 0) (type default))
@@
     (stroke (width 0) (type default))
   )
+  (wire (pts (xy 63.5 39.37) (xy 63.5 40.64))
+    (stroke (width 0) (type default))
+  )
   (wire (pts (xy 153.67 114.3) (xy 161.29 114.3))
     (stroke (width 0) (type default))
@@
     (stroke (width 0) (type default))
   )
+  (wire (pts (xy 33.02 33.02) (xy 38.1 33.02))
+    (stroke (width 0) (type default))
+  )
   (wire (pts (xy 157.48 129.54) (xy 157.48 132.08))
     (stroke (width 0) (type default))
@@
     (stroke (width 0) (type default))
   )
-  (wire (pts (xy 123.19 38.1) (xy 123.19 43.18))
+  (wire (pts (xy 123.19 38.1) (xy 123.19 39.37))
     (stroke (width 0) (type default))
   )
@@
     (stroke (width 0) (type default))
   )
+  (wire (pts (xy 33.02 39.37) (xy 33.02 40.64))
+    (stroke (width 0) (type default))
+  )
   (wire (pts (xy 242.57 33.02) (xy 251.46 33.02))
     (stroke (width 0) (type default))
@@
     (stroke (width 0) (type default))
   )
+  (wire (pts (xy 63.5 33.02) (xy 58.42 33.02))
+    (stroke (width 0) (type default))
+  )
   (wire (pts (xy 161.29 99.06) (xy 172.085 99.06))
     (stroke (width 0) (type default))
@@
     (stroke (width 0) (type default))
   )
+  (wire (pts (xy 33.02 40.64) (xy 38.1 40.64))
+    (stroke (width 0) (type default))
+  )
   (wire (pts (xy 34.29 144.78) (xy 41.91 144.78))
     (stroke (width 0) (type default))
@@
     (stroke (width 0) (type default))
   )
+  (wire (pts (xy 63.5 34.29) (xy 63.5 33.02))
+    (stroke (width 0) (type default))
+  )
   (wire (pts (xy 38.1 40.64) (xy 45.72 40.64))
     (stroke (width 0) (type default))
@@
     (stroke (width 0) (type default))
   )
+  (wire (pts (xy 123.19 39.37) (xy 123.19 43.18))
+    (stroke (width 0) (type default))
+  )
   (wire (pts (xy 212.09 76.2) (xy 214.63 76.2))
     (stroke (width 0) (type default))
@@
     (stroke (width 0) (type default))
   )
+  (wire (pts (xy 130.81 39.37) (xy 133.35 39.37))
+    (stroke (width 0) (type default))
+  )
   (wire (pts (xy 190.5 33.02) (xy 199.39 33.02))
     (stroke (width 0) (type default))
@@
     (stroke (width 0) (type default))
   )
+  (wire (pts (xy 33.02 34.29) (xy 33.02 33.02))
+    (stroke (width 0) (type default))
+  )
   (wire (pts (xy 161.29 96.52) (xy 172.085 96.52))
     (stroke (width 0) (type default))
@@
   )
   (wire (pts (xy 155.067 142.24) (xy 157.48 142.24))
+    (stroke (width 0) (type default))
+  )
+  (wire (pts (xy 63.5 40.64) (xy 58.42 40.64))
     (stroke (width 0) (type default))
   )
@@
     (effects (font (size 1.27 1.27)) (justify left bottom))
   )
-  (label "GP04" (at 233.68 132.08 180) (fields_autoplaced)
+  (label "GP10" (at 233.68 132.08 180) (fields_autoplaced)
     (effects (font (size 1.27 1.27) bold) (justify right bottom))
   )
@@
     (effects (font (size 0.8 0.8) bold) (justify right bottom))
   )
-  (label "GP08" (at 62.23 144.78 0) (fields_autoplaced)
+  (label "GP04" (at 62.23 144.78 0) (fields_autoplaced)
     (effects (font (size 1.27 1.27) bold) (justify left bottom))
   )
@@
     (effects (font (size 1.27 1.27) (thickness 0.254) bold) (justify right bottom))
   )
-  (label "GP10" (at 62.23 139.7 0) (fields_autoplaced)
+  (label "GP08" (at 62.23 139.7 0) (fields_autoplaced)
     (effects (font (size 1.27 1.27) bold) (justify left bottom))
   )
@@
     )
   )
+  (symbol (lib_id "Device:C_Polarized_Small") (at 33.02 36.83 0) (mirror y) (unit 1)
+    (in_bom yes) (on_board yes) (dnp no)
+    (property "Reference" "C3" (at 30.48 35.56 0)
+      (effects (font (size 1.27 1.27)) (justify left))
+    )
+    (property "Value" "C_pth" (at 31.75 39.37 0)
+      (effects (font (size 1.27 1.27)) (justify left))
+    )
+    (property "Footprint" "Capacitor_THT:CP_Radial_D5.0mm_P2.50mm" (at 33.02 36.83 0)
+      (effects (font (size 1.27 1.27)) hide)
+    )
+    (property "Datasheet" "~" (at 33.02 36.83 0)
+      (effects (font (size 1.27 1.27)) hide)
+    )
+    (property "partnumber" "" (at 33.02 36.83 0)
+      (effects (font (size 1.27 1.27)) hide)
+    )
+    (pin "1")
+    (pin "2")
+    (instances
+      (project "bitdoglab_v5"
+        (path "/09159d3e-7c55-4754-a166-a35b245d09f3"
+          (reference "C3") (unit 1)
+        )
+      )
+    )
+  )
   (symbol (lib_id "Raspberry_Pi_Pico_W_SC0918:DMG2305UX-13") (at 120.65 30.48 90) (unit 1)
     (in_bom yes) (on_board yes) (dnp no) (fields_autoplaced)
@@
     )
   )
+  (symbol (lib_id "Device:C_Polarized_Small") (at 63.5 36.83 0) (unit 1)
+    (in_bom yes) (on_board yes) (dnp no)
+    (property "Reference" "C4" (at 66.04 35.0139 0)
+      (effects (font (size 1.27 1.27)) (justify left))
+    )
+    (property "Value" "C_pth" (at 66.04 37.5539 0)
+      (effects (font (size 1.27 1.27)) (justify left))
+    )
+    (property "Footprint" "Capacitor_THT:CP_Radial_D5.0mm_P2.50mm" (at 63.5 36.83 0)
+      (effects (font (size 1.27 1.27)) hide)
+    )
+    (property "Datasheet" "~" (at 63.5 36.83 0)
+      (effects (font (size 1.27 1.27)) hide)
+    )
+    (property "partnumber" "" (at 63.5 36.83 0)
+      (effects (font (size 1.27 1.27)) hide)
+    )
+    (pin "1")
+    (pin "2")
+    (instances
+      (project "bitdoglab_v5"
+        (path "/09159d3e-7c55-4754-a166-a35b245d09f3"
+          (reference "C4") (unit 1)
+        )
+      )
+    )
+  )
   (symbol (lib_id "Device:C_Polarized_Small") (at 38.1 36.83 0) (mirror y) (unit 1)
     (in_bom yes) (on_board yes) (dnp no)
-    (property "Reference" "C1" (at 35.56 35.0139 0)
+    (property "Reference" "C1" (at 38.1 34.29 0)
       (effects (font (size 1.27 1.27)) (justify left))
     )
-    (property "Value" "C_Polarized_Small" (at 35.56 37.5539 0)
+    (property "Value" "C_smd" (at 40.64 39.37 0)
       (effects (font (size 1.27 1.27)) (justify left))
     )
@@
     )
   )
+  (symbol (lib_id "power:GNDREF") (at 133.35 39.37 90) (unit 1)
+    (in_bom yes) (on_board yes) (dnp no)
+    (property "Reference" "#PWR027" (at 139.7 39.37 0)
+      (effects (font (size 1.27 1.27)) hide)
+    )
+    (property "Value" "GNDREF" (at 135.89 44.45 0)
+      (effects (font (size 1.27 1.27)) hide)
+    )
+    (property "Footprint" "" (at 133.35 39.37 0)
+      (effects (font (size 1.27 1.27)) hide)
+    )
+    (property "Datasheet" "" (at 133.35 39.37 0)
+      (effects (font (size 1.27 1.27)) hide)
+    )
+    (pin "1")
+    (instances
+      (project "bitdoglab_v5"
+        (path "/09159d3e-7c55-4754-a166-a35b245d09f3"
+          (reference "#PWR027") (unit 1)
+        )
+      )
+    )
+  )
   (symbol (lib_id "Connector_custom:Conn_01x02") (at 252.73 29.21 0) (unit 1)
     (in_bom yes) (on_board yes) (dnp no) (fields_autoplaced)
@@
   (symbol (lib_id "Device:C_Polarized_Small") (at 58.42 36.83 0) (unit 1)
     (in_bom yes) (on_board yes) (dnp no)
-    (property "Reference" "C2" (at 60.96 35.0139 0)
+    (property "Reference" "C2" (at 54.61 34.29 0)
       (effects (font (size 1.27 1.27)) (justify left))
     )
-    (property "Value" "C_Polarized_Small" (at 60.96 37.5539 0)
+    (property "Value" "C_smd" (at 55.88 40.64 0)
       (effects (font (size 1.27 1.27)) (justify left))
     )
@@
   (symbol (lib_id "Raspberry_Pi_Pico_W_SC0918:SC0918") (at 186.69 107.95 0) (unit 1)
     (in_bom yes) (on_board yes) (dnp no) (fields_autoplaced)
-    (property "Reference" "A1" (at 186.69 54.61 0)
+    (property "Reference" "pico1" (at 186.69 54.61 0)
       (effects (font (size 1.27 1.27)))
     )
@@
       (project "bitdoglab_v5"
         (path "/09159d3e-7c55-4754-a166-a35b245d09f3"
-          (reference "A1") (unit 1)
+          (reference "pico1") (unit 1)
         )
       )
@@
         )
       )
+    )
+  )
+  (symbol (lib_id "Device:R") (at 127 39.37 90) (unit 1)
+    (in_bom yes) (on_board yes) (dnp no)
+    (property "Reference" "R_pulldown1" (at 129.54 40.64 90)
+      (effects (font (size 1.27 1.27)))
+    )
+    (property "Value" "10k" (at 129.54 36.83 90)
+      (effects (font (size 1.27 1.27)))
+    )
+    (property "Footprint" "Resistor_THT:R_Axial_DIN0207_L6.3mm_D2.5mm_P7.62mm_Horizontal" (at 127 41.148 90)
+      (effects (font (size 1.27 1.27)) hide)
+    )
+    (property "Datasheet" "~" (at 127 39.37 0)
+      (effects (font (size 1.27 1.27)) hide)
+    )
+    (property "partnumber" "" (at 127 39.37 0)
+      (effects (font (size 1.27 1.27)) hide)
+    )
+    (pin "1")
+    (pin "2")
+    (instances
+      (project "bitdoglab_v5"
+        (path "/09159d3e-7c55-4754-a166-a35b245d09f3"
+          (reference "R_pulldown1") (unit 1)
+        )
+      )
